File: rpi_breakout.kicad_pcb (KiCad board)
At the start: 2 copper layers, 41 parts, among them J1 USB4520-03-0-A, J2 Conn_01x10, J3 Conn_01x10, U1 SC0914_13_, U2 W25Q16JVZPIQ, U3 AP2112K-3.3TRG1, Y1 ABM8-12.000MHZ-B2-T

Commit message: Routing
Parts:
- removed C3: 100nF, Capacitor_SMD:C_0402_1005Metric
- BOOTSEL1, C1, C10, C11, C12, C16, C2, C4, C5, C6, C7, C8, C9, D1, D_POWER1, J1, J2, J3, J_SWD1, R1, R12, R13, R2, R3, R4, R5, R6, R7, R8, R9, RESET1: moved to B.Cu
- moved J2 46.6 mm to (174.9, 50.9)
- moved J_SWD1 45.6 mm to (151.8, 66.4)
- moved C13 43.3 mm to (176.1, 63.3), turned to -90 degrees
- moved J3 37.5 mm to (174.9, 71.1)
- moved R12 34.4 mm to (155.7, 66.3), turned to 180 degrees
- moved D_POWER1 33.5 mm to (155.3, 68.0), turned to 180 degrees
- moved R11 31.7 mm to (177.5, 56.4)
- moved BOOTSEL1 30.2 mm to (156.8, 56.5), turned to 180 degrees
- moved R8 30.1 mm to (174.8, 56.5)
- moved RESET1 29.8 mm to (156.7, 62.7), turned to 180 degrees
- moved R10 29.1 mm to (174.9, 63.3), turned to 90 degrees
- moved R13 28.0 mm to (160.0, 66.3), turned to 180 degrees
- moved D1 26.9 mm to (159.6, 68.0), turned to 180 degrees
- moved R6 26.8 mm to (172.3, 59.0)
- moved U2 25.3 mm to (174.2, 58.7), turned to -90 degrees
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Routing:
- net VBUS: track 0.00 -> 40.7 mm, vias 0 -> 1
- net +3.3V: track 0.00 -> 29.9 mm, vias 0 -> 3
- net /GPIO23: track 0.00 -> 12.9 mm
- net /GPIO24: track 0.00 -> 11.9 mm
- net /GPIO9: track 0.00 -> 11.8 mm
- net /GPIO0: track 0.00 -> 11.3 mm
- net /GPIO25: track 0.00 -> 11.0 mm
- net /ADC3: track 0.00 -> 10.9 mm
- net /SWDIO: track 0.00 -> 10.3 mm
- net /ADC0: track 0.00 -> 10.2 mm
- net /ADC2: track 0.00 -> 9.99 mm
- net /GPIO8: track 0.00 -> 9.94 mm
- net Net-(U1-USB_DP): track 0.00 -> 9.44 mm, vias 0 -> 1
- net /SWCLK: track 0.00 -> 9.43 mm
- net Net-(U1-RUN): track 0.00 -> 9.35 mm, vias 0 -> 1
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- added copper zone on In2.Cu, net +3.3V
- added copper zone on B.Cu, net GND
- added copper zone on F.Cu, net GND
- added copper zone on In1.Cu, net GND
Other:
- board outline added: 36.8 x 24.1 mm
- copper layers 2 -> 4
