File: rpi_breakout.kicad_sch (KiCad schematic)
At the start: 13 parts, among them J1 USB4520-03-0-A, J2 Conn_01x10, U1 SC0914_13_, U2 W25Q16JVZPIQ, U3 AP2112K-3.3TRG1, Y1 ABM8-12.000MHZ-B2-T

Commit message: Schematic updates; Starting pcb
Parts:
- added C1, C10, C13, C2, C3, C4, C5, C6, C7, C8: 100nF, Capacitor_SMD:C_0402_1005Metric, symbol Device:C_Small
- added C11, C12, C16, C9: 1uF, Capacitor_SMD:C_0402_1005Metric, symbol Device:C_Small
- added C14, C15: 27pF, Capacitor_SMD:C_0402_1005Metric, symbol Device:C_Small
- added D1, D_POWER1: LED, LED_SMD:LED_0805_2012Metric, symbol Device:LED
- added J3: Conn_01x10, Connector_PinHeader_2.54mm:PinHeader_1x10_P2.54mm_Vertical, symbol Connector_Generic:Conn_01x10
- added J_SWD1: Conn_01x04, Connector_PinHeader_2.54mm:PinHeader_1x04_P2.54mm_Vertical, symbol Connector_Generic:Conn_01x04
- added R10, R11, R6, R7, R8, R9: 10k, Resistor_SMD:R_0402_1005Metric, symbol Device:R_Small_US
- added R12, R13: 68, Resistor_SMD:R_0402_1005Metric, symbol Device:R_Small_US
- BOOTSEL1: renamed from BOOTSEL; footprint SKRWAEE030 -> KiCad:SKRWAEE030
- J1: footprint USB4520030A -> KiCad_USB:USB4520030A
- J2: footprint (none) -> Connector_PinHeader_2.54mm:PinHeader_1x10_P2.54mm_Vertical
- R1, R2, R3, R4, R5: footprint (none) -> Resistor_SMD:R_0402_1005Metric
- RESET1: renamed from RESET; footprint SKRWAEE030 -> KiCad:SKRWAEE030
- U3: footprint AP2112K-3.3TRG1:SOT95P285X140-5N -> AP2112K_3_3TRG1:SOT95P285X140-5N
- Y1: footprint ABM8-12.000MHZ-B2-T:XTAL_ABM8-12.000MHZ-B2-T -> ABM8_12_000MHZ_B2_T:XTAL_ABM8-12.000MHZ-B2-T
Connections:
- net +3.3V: now also C1.1, C10.1, C12.1, C13.1, C16.2, C2.1, C3.1, C4.1, C5.1, C6.1, C7.1, C8.1, D1.2 (A), D_POWER1.2 (A), J3.2 (Pin_2), J_SWD1.1 (Pin_1), R10.1, R11.1, R6.1, R7.1, R8.1, R9.1
- net GND: now also J1.MH1, J1.MH2, J1.MH3, J1.MH4, C1.2, C10.2, C11.2, C12.2, C13.2, C14.2, C15.1, C16.1, C2.2, C3.2, C4.2, C5.2, C6.2, C7.2, C8.2, C9.2, J3.1 (Pin_1), J_SWD1.4 (Pin_4), R12.2
- net VBUS: now also C11.1, J3.10 (Pin_10)
- net at U1.20 (XIN), Y1.1: now also C15.2
- net at U1.21 (XOUT), Y1.3: now also C14.1
- net QSPI_SS_N: now reaches BOOTSEL1.2, BOOTSEL1.4, U1.56 (QSPI_SS_N), U2.1 (~{CS})
- net QSPI_SS_N: now also R11.2
- net QSPI_SD1: now reaches U1.55 (QSPI_SD1), U2.2 (DO(IO1))
- net QSPI_SD1: now also R8.2
- net QSPI_SD2: now reaches U1.54 (QSPI_SD2), U2.3 (~{WP}(IO2))
- net QSPI_SD2: now also R9.2
- net QSPI_SD0: now reaches U1.53 (QSPI_SD0), U2.5 (DI(IO0))
- net QSPI_SD0: now also R7.2
- net QSPI_SCLK: now reaches U1.52 (QSPI_SCLK), U2.6 (CLK)
- net QSPI_SCLK: now also R6.2
- net QSPI_SD3: now reaches U1.51 (QSPI_SD3), U2.7 (~{HOLD}/RESET(IO3))
- net QSPI_SD3: now also R10.2
- net GPIO0: now reaches J2.1 (Pin_1)
- net GPIO0: now also U1.2 (GPIO0); no longer U1.9 (GPIO7)
- net GPIO9: now reaches J2.10 (Pin_10)
- net GPIO9: now also U1.12 (GPIO9); no longer U1.24 (SWCLK)
- net GPIO1: now reaches J2.2 (Pin_2)
- net GPIO1: now also U1.3 (GPIO1); no longer U1.8 (GPIO6)
- net GPIO2: now reaches J2.3 (Pin_3)
- net GPIO2: now also U1.4 (GPIO2); no longer U1.7 (GPIO5)
- net GPIO3: now reaches J2.4 (Pin_4)
- net GPIO3: now also U1.5 (GPIO3); no longer U1.6 (GPIO4)
- net GPIO4: now reaches J2.5 (Pin_5)
- net GPIO4: now also U1.6 (GPIO4); no longer U1.5 (GPIO3)
- net GPIO5: now reaches J2.6 (Pin_6)
- net GPIO5: now also U1.7 (GPIO5); no longer U1.4 (GPIO2)
- net GPIO6: now reaches J2.7 (Pin_7)
- net GPIO6: now also U1.8 (GPIO6); no longer U1.3 (GPIO1)
- net GPIO7: now reaches J2.8 (Pin_8)
- net GPIO7: now also U1.9 (GPIO7); no longer U1.2 (GPIO0)
- net GPIO8: now reaches J2.9 (Pin_9)
- net GPIO8: now also U1.11 (GPIO8); no longer U1.25 (SWDIO)
- net GPIO15: now reaches U1.18 (GPIO15)
- net GPIO15: now also R13.2
- net V_REG: now reaches U1.23 (DVDD), U1.45 (VREG_VOUT), U1.50 (DVDD__1)
- net V_REG: now also C9.1
- net GPIO23: now reaches U1.35 (GPIO23)
- net GPIO23: now also J3.9 (Pin_9)
- net GPIO24: now reaches U1.36 (GPIO24)
- net GPIO24: now also J3.8 (Pin_8)
- net GPIO25: now reaches U1.37 (GPIO25)
- net GPIO25: now also J3.7 (Pin_7)
- net ADC0: now reaches U1.38 (GPIO26/ADC0)
- net ADC0: now also J3.6 (Pin_6)
- net ADC1: now reaches U1.39 (GPIO27/ADC1)
- net ADC1: now also J3.5 (Pin_5)
- net ADC2: now reaches U1.40 (GPIO28/ADC2)
- net ADC2: now also J3.4 (Pin_4)
- net ADC3: now reaches U1.41 (GPIO29/ADC3)
- net ADC3: now also J3.3 (Pin_3)
- new net: D_POWER1.1 (K), R12.1
- new net: D1.1 (K), R13.1
- new net SWCLK: J_SWD1.3 (Pin_3), U1.24 (SWCLK)
- new net SWDIO: J_SWD1.2 (Pin_2), U1.25 (SWDIO)
Other:
- moved on the sheet: BOOTSEL1, U2

Commit message: Routing
Parts:
- removed C3: 100nF, Capacitor_SMD:C_0402_1005Metric, symbol Device:C_Small
Changed lines of the file:
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@@
 	(wire
 		(pts
-			(xy 74.93 21.59) (xy 74.93 26.67)
-		)
-		(stroke
-			(width 0)
-			(type default)
-		)
-	)
-	(wire
-		(pts
 			(xy 142.24 21.59) (xy 153.67 21.59)
 		)
@@
 	)
 	(symbol
-		(lib_id "Device:C_Small")
-		(at 74.93 29.21 0)
-		(unit 1)
-		(exclude_from_sim no)
-		(in_bom yes)
-		(on_board yes)
-		(dnp no)
-		(fields_autoplaced yes)
-		(property "Reference" "C3"
-			(at 77.47 27.9462 0)
-			(effects
-				(font
-					(size 1.27 1.27)
-				)
-				(justify left)
-			)
-		)
-		(property "Value" "100nF"
-			(at 77.47 30.4862 0)
-			(effects
-				(font
-					(size 1.27 1.27)
-				)
-				(justify left)
-			)
-		)
-		(property "Footprint" "Capacitor_SMD:C_0402_1005Metric"
-			(at 74.93 29.21 0)
-			(effects
-				(font
-					(size 1.27 1.27)
-				)
-				(hide yes)
-			)
-		)
-		(property "Datasheet" "~"
-			(at 74.93 29.21 0)
-			(effects
-				(font
-					(size 1.27 1.27)
-				)
-				(hide yes)
-			)
-		)
-		(property "Description" "Unpolarized capacitor, small symbol"
-			(at 74.93 29.21 0)
-			(effects
-				(font
-					(size 1.27 1.27)
-				)
-				(hide yes)
-			)
-		)
-		(pin "1"
-		)
-		(pin "2"
-		)
-		(instances
-			(project "rpi_breakout"
-				(path "/e6e76701-c43e-4a4c-9916-d31d8a705258"
-					(reference "C3")
-					(unit 1)
-				)
-			)
-		)
-	)
-	(symbol
 		(lib_id "power:GND")
 		(at 57.15 53.34 180)
@@
 	)
 	(symbol
-		(lib_id "power:GND")
-		(at 74.93 31.75 0)
-		(unit 1)
-		(exclude_from_sim no)
-		(in_bom yes)
-		(on_board yes)
-		(dnp no)
-		(fields_autoplaced yes)
-		(property "Reference" "#PWR034"
-			(at 74.93 38.1 0)
-			(effects
-				(font
-					(size 1.27 1.27)
-				)
-				(hide yes)
-			)
-		)
-		(property "Value" "GND"
-			(at 74.93 36.83 0)
-			(effects
-				(font
-					(size 1.27 1.27)
-				)
-			)
-		)
-		(property "Footprint" ""
-			(at 74.93 31.75 0)
-			(effects
-				(font
-					(size 1.27 1.27)
-				)
-				(hide yes)
-			)
-		)
-		(property "Datasheet" ""
-			(at 74.93 31.75 0)
-			(effects
-				(font
-					(size 1.27 1.27)
-				)
-				(hide yes)
-			)
-		)
-		(property "Description" "Power symbol creates a global label with name \"GND\" , ground"
-			(at 74.93 31.75 0)
-			(effects
-				(font
-					(size 1.27 1.27)
-				)
-				(hide yes)
-			)
-		)
-		(pin "1"
-		)
-		(instances
-			(project ""
-				(path "/e6e76701-c43e-4a4c-9916-d31d8a705258"
-					(reference "#PWR034")
-					(unit 1)
-				)
-			)
-		)
-	)
-	(symbol
 		(lib_id "Device:R_Small_US")
 		(at 259.08 22.86 90)
@@
 					(unit 1)
 				)
-			)
-		)
-	)
-	(symbol
-		(lib_id "power:+3.3V")
-		(at 74.93 21.59 0)
-		(unit 1)
-		(exclude_from_sim no)
-		(in_bom yes)
-		(on_board yes)
-		(dnp no)
-		(fields_autoplaced yes)
-		(property "Reference" "#PWR016"
-			(at 74.93 25.4 0)
-			(effects
-				(font
-					(size 1.27 1.27)
-				)
-				(hide yes)
-			)
-		)
-		(property "Value" "+3.3V"
-			(at 74.93 16.51 0)
-			(effects
-				(font
-					(size 1.27 1.27)
-				)
-			)
-		)
-		(property "Footprint" ""
-			(at 74.93 21.59 0)
-			(effects
-				(font
-					(size 1.27 1.27)
-				)
-				(hide yes)
-			)
-		)
-		(property "Datasheet" ""
-			(at 74.93 21.59 0)
-			(effects
-				(font
-					(size 1.27 1.27)
-				)
-				(hide yes)
-			)
-		)
-		(property "Description" "Power symbol creates a global label with name \"+3.3V\""
-			(at 74.93 21.59 0)
-			(effects
-				(font
-					(size 1.27 1.27)
-				)
-				(hide yes)
-			)
-		)
-		(pin "1"
-		)
-		(instances
-			(project ""
-				(path "/e6e76701-c43e-4a4c-9916-d31d8a705258"
-					(reference "#PWR016")
-					(unit 1)
-				)
